Commit message: Add files via upload

File: delirobot_description/urdf/delirobot.xacro (robot description, xacro)
@@ -22,13 +22,4 @@
             </geometry>
         </collision>
-        <!-- <visual name='chassis_visual'>
-            <origin xyz="0 0 0" rpy=" 0 0 0"/>
-            <geometry>
-                <box size=".1 .1 .1"/>
-            </geometry>
-            <material name="">
-                <color rgba="1 1 1 1" />
-            </material>
-        </visual> -->
         <collision name='back_caster_collision'>
             <origin xyz="-0.1 0 -0.05" rpy=" 0 0 0"/>
